Commit message: Mod_180

File: src/rubot_mecanum_description/urdf/rubot_bueno.urdf (robot description, URDF)
Before this commit: robot nexus, 8 links, 7 joints
Links:
- link base_scan: geometry collision cylinder length=0.01575 radius=0.0275; visual mesh filename=package://rubot_mecanum_description/meshes/rubot/lidar.stl scale=0.001 0.001 0.001
Joints:
- joint scan_joint: origin xyz=0 0 0.09 rpy=0 0 3.14 -> xyz=0.111 0.076 0.124 rpy=0 0 3.14
