Commit message: ArreglandoNexus

File: src/rubot_mecanum_description/urdf/rubot.urdf (robot description, URDF)
Before this commit: robot nexus, 8 links, 7 joints
Joints:
- joint scan_joint: origin xyz=0.111 0.076 0.124 rpy=0 0 3.14 -> xyz=0.111 0.076 0.124 rpy=0 0 0

Commit message: rubot_funciona_laberinto

File: src/rubot_mecanum_description/urdf/rubot.urdf (robot description, URDF)
Before this commit: robot nexus, 8 links, 7 joints
Links:
- link base_link: mass 10 -> 2
- link lower_left_wheel: mass 0.3844 -> 0.05
- link lower_right_wheel: mass 0.3844 -> 0.05
- link upper_left_wheel: mass 0.3844 -> 0.05
- link upper_right_wheel: mass 0.3844 -> 0.05
Joints:
- joint scan_joint: origin xyz=0.111 0.076 0.124 rpy=0 0 0 -> xyz=0.111 0.076 0.124 rpy=0 0 3.14
